Commit message: v2.8.0

File: rsc/motorOperatingRegion/quadruped_rig.urdf (robot description, URDF)
Before this commit: robot mor_quadruped_rig, 14 links, 13 joints
Joints:
- joint LF_HAA: limit lower=-0.6 upper=0.6 effort=18 -> lower=-0.6 upper=0.6 effort=18 velocity=60
- joint LF_HFE: limit effort=30 -> effort=30 velocity=36
- joint LF_KFE: limit effort=30 -> effort=30 velocity=36
- joint LH_HAA: limit lower=-0.6 upper=0.6 effort=18 -> lower=-0.6 upper=0.6 effort=18 velocity=60
- joint LH_HFE: limit effort=30 -> effort=30 velocity=36
- joint LH_KFE: limit effort=30 -> effort=30 velocity=36
- joint RF_HAA: limit lower=-0.6 upper=0.6 effort=18 -> lower=-0.6 upper=0.6 effort=18 velocity=60
- joint RF_HFE: limit effort=30 -> effort=30 velocity=36
- joint RF_KFE: limit effort=30 -> effort=30 velocity=36
- joint RH_HAA: limit lower=-0.6 upper=0.6 effort=18 -> lower=-0.6 upper=0.6 effort=18 velocity=60
- joint RH_HFE: limit effort=30 -> effort=30 velocity=36
- joint RH_KFE: limit effort=30 -> effort=30 velocity=36
